Commit message: Put left leg kneeling position

File: urdf/darwin.urdf (robot description, URDF)
Before this commit: robot darwinOP, 31 links, 30 joints
Joints:
- joint j_ankle1_l: origin xyz=-0.093 0 0 rpy=3.14159 0 0 -> xyz=-0.093 0 0 rpy=3.14159 0 1.1288
- joint j_thigh2_l: origin xyz=0 0 0 rpy=1.5707963 0 -1.5707963 -> xyz=0 0 0 rpy=1.5707963 -1.122 -1.5707963
- joint j_tibia_l: origin xyz=-0.093 0 0 rpy=0 0 0 -> xyz=-0.093 0 0 rpy=0 0 -2.26

Commit message: Enhance left kneeling position

File: urdf/darwin.urdf (robot description, URDF)
Before this commit: robot darwinOP, 31 links, 30 joints
Joints:
- joint j_ankle1_l: origin xyz=-0.093 0 0 rpy=3.14159 0 1.1288 -> xyz=-0.093 0 0 rpy=3.14159 0 1.1388
- joint j_thigh2_l: origin xyz=0 0 0 rpy=1.5707963 -1.122 -1.5707963 -> xyz=0 0 0 rpy=1.5707963 -1.142 -1.5707963
- joint j_tibia_l: origin xyz=-0.093 0 0 rpy=0 0 -2.26 -> xyz=-0.093 0 0 rpy=0 0 -2.2788

Commit message: Complete legs kneeling position

File: urdf/darwin.urdf (robot description, URDF)
Before this commit: robot darwinOP, 31 links, 30 joints
Joints:
- joint j_ankle1_r: origin xyz=0.093 0 0 rpy=3.14159 0 0 -> xyz=0.093 0 0 rpy=3.14159 0 -1.1388
- joint j_thigh2_r: origin xyz=0 0 0 rpy=1.5707963 0 -1.5707963 -> xyz=0 0 0 rpy=1.5707963 1.142 -1.5707963
- joint j_tibia_r: origin xyz=0.093 0 0 rpy=0 0 0 -> xyz=0.093 0 0 rpy=0 0 2.2788

Commit message: Move left arm into starting position

File: urdf/darwin.urdf (robot description, URDF)
Before this commit: robot darwinOP, 31 links, 30 joints
Joints:
- joint j_high_arm_l: origin xyz=-0.016 0 0.02165 rpy=1.5707963 1.5707963 0 -> xyz=-0.016 0 0.02165 rpy=1.5707963 0.2 0
- joint j_low_arm_l: origin xyz=-0.06 0 -0.016 rpy=-1.5707963 3.14159 0 -> xyz=-0.06 0 -0.016 rpy=-1.5707963 1.64159 0
- joint j_shoulder_l: origin xyz=0 0 0 rpy=0 0 -1.5707963 -> xyz=0 0 0 rpy=0 0 -1.15

Commit message: Move right arm into starting position

File: urdf/darwin.urdf (robot description, URDF)
Before this commit: robot darwinOP, 31 links, 30 joints
Joints:
- joint j_high_arm_r: origin xyz=0.016 0 0.02165 rpy=-1.5707963 1.5707963 0 -> xyz=0.016 0 0.02165 rpy=-1.5707963 2.9415926 0
- joint j_low_arm_r: origin xyz=-0.06 0 0.016 rpy=-1.5707963 3.14159 0 -> xyz=-0.06 0 0.016 rpy=-1.5707963 4.64159 0
- joint j_shoulder_r: origin xyz=0 0 0 rpy=0 0 -1.5707963 -> xyz=0 0 0 rpy=0 0 -1.9907

Commit message: Update inertia matrix

File: urdf/darwin.urdf (robot description, URDF)
Before this commit: robot darwinOP, 31 links, 30 joints
Links:
- link MP_PELVIS_L: mass 0.167 -> 0.167108
- link MP_PELVIS_R: mass 0.197 -> 0.167108

Commit message: Update inertia parameters for MP_NECK

File: urdf/darwin.urdf (robot description, URDF)
Before this commit: robot darwinOP, 31 links, 30 joints
Links:
- link MP_NECK: mass 0.024357719 -> 0.02435772

Commit message: Update inertia paramentes for MP_SHOULDER_L

File: urdf/darwin.urdf (robot description, URDF)
Before this commit: robot darwinOP, 31 links, 30 joints
Links:
- link MP_SHOULDER_L: mass 0.025913024 -> 0.02591302

Commit message: Update inertia paramentes for MP_SHOULDER_R

File: urdf/darwin.urdf (robot description, URDF)
Before this commit: robot darwinOP, 31 links, 30 joints
Links:
- link MP_SHOULDER_R: mass 0.025913024 -> 0.02591302

Commit message: Update inertia paramenters for MP_TIBIA_L

File: urdf/darwin.urdf (robot description, URDF)
Before this commit: robot darwinOP, 31 links, 30 joints
Links:
- link MP_TIBIA_L: mass 0.070309794 -> 0.07030979

Commit message: Update inertia paramenters for MP_TIBIA_R

File: urdf/darwin.urdf (robot description, URDF)
Before this commit: robot darwinOP, 31 links, 30 joints
Links:
- link MP_TIBIA_R: mass 0.070309794 -> 0.07030979

Commit message: Update inertia parameters for MP_BACK_L

File: urdf/darwin.urdf (robot description, URDF)
Before this commit: robot darwinOP, 31 links, 30 joints
Links:
- link MP_BACK_L: mass 0.010 -> 0.01

Commit message: Update inertia parameters for MP_BACK_R

File: urdf/darwin.urdf (robot description, URDF)
Before this commit: robot darwinOP, 31 links, 30 joints
Links:
- link MP_BACK_R: mass 0.010 -> 0.01

Commit message: Update inertial paramenters for MP_ARM_LOW_L

File: urdf/darwin.urdf (robot description, URDF)
Before this commit: robot darwinOP, 31 links, 30 joints
Links:
- link MP_ARM_LOW_L: mass 0.059288504 -> 0.0592885

Commit message: Update inertia paramaters for MP_ARM_GRIPPER_FIX_DUMMY_L

File: urdf/darwin.urdf (robot description, URDF)
Before this commit: robot darwinOP, 31 links, 30 joints
Links:
- link MP_ARM_GRIPPER_FIX_DUMMY_L: mass 0.010 -> 0.01

Commit message: Update inertia paramenters for MP_ARM_GRIPPER_MOV_L

File: urdf/darwin.urdf (robot description, URDF)
Before this commit: robot darwinOP, 31 links, 30 joints
Links:
- link MP_ARM_GRIPPER_MOV_L: mass 0.010 -> 0.01

Commit message: Update inertia parameters for MP_ARM_GRIPPER_FIX_L

File: urdf/darwin.urdf (robot description, URDF)
Before this commit: robot darwinOP, 31 links, 30 joints
Links:
- link MP_ARM_GRIPPER_FIX_L: mass 0.010 -> 0.01

Commit message: Update inertia paramenters for MP_ARM_GRIPPER_FIX_R

File: urdf/darwin.urdf (robot description, URDF)
Before this commit: robot darwinOP, 31 links, 30 joints
Links:
- link MP_ARM_GRIPPER_FIX_R: mass 0.010 -> 0.01

Commit message: Update inertia parameters for MP_ARM_GRIPPER_FIX_DUMMY_R

File: urdf/darwin.urdf (robot description, URDF)
Before this commit: robot darwinOP, 31 links, 30 joints
Links:
- link MP_ARM_GRIPPER_FIX_DUMMY_R: mass 0.010 -> 0.01

Commit message: Update inertia paramenter for MP_ARM_GRIPPER_MOV_R

File: urdf/darwin.urdf (robot description, URDF)
Before this commit: robot darwinOP, 31 links, 30 joints
Links:
- link MP_ARM_GRIPPER_MOV_R: mass 0.010 -> 0.01

Commit message: Update inertia parameters for MP_ARM_LOW_R

File: urdf/darwin.urdf (robot description, URDF)
Before this commit: robot darwinOP, 31 links, 30 joints
Links:
- link MP_ARM_LOW_R: mass 0.059288504 -> 0.0592885

Commit message: Update lower and upper limits for j_tilt

File: urdf/darwin.urdf (robot description, URDF)
Before this commit: robot darwinOP, 31 links, 30 joints
Joints:
- joint j_tilt: limit lower=-2.6179939 upper=2.6179939 effort=2.8 velocity=5.6548668 -> lower=-1.0471976 upper=0.5235988 effort=2.8 velocity=5.6548668

Commit message: Update lower and upper limits for j_shoulder_l (shoulder pitch)

File: urdf/darwin.urdf (robot description, URDF)
Before this commit: robot darwinOP, 31 links, 30 joints
Joints:
- joint j_shoulder_l: limit lower=-2.6179939 upper=2.6179939 effort=2.8 velocity=5.6548668 -> lower=-4.3633231 upper=4.3633231 effort=2.8 velocity=5.6548668

Commit message: Update lower and upper limits for j_high_arm_l (shoulder roll)

File: urdf/darwin.urdf (robot description, URDF)
Before this commit: robot darwinOP, 31 links, 30 joints
Joints:
- joint j_high_arm_l: limit lower=-2.6179939 upper=2.6179939 effort=2.8 velocity=5.648668 -> lower=-1.7453293 upper=1.7453293 effort=2.8 velocity=5.648668

Commit message: Update lower and upper limits for j_low_arm_l (elbow)

File: urdf/darwin.urdf (robot description, URDF)
Before this commit: robot darwinOP, 31 links, 30 joints
Joints:
- joint j_low_arm_l: limit lower=-2.6179939 upper=2.6179939 effort=2.8 velocity=5.6548668 -> lower=-2.7925268 upper=0 effort=2.8 velocity=5.6548668

Commit message: Update lower and upper limits for j_gripper_l
This is not based on the article because this joint is not described. I
used rviz to visually choose a proper value.

File: urdf/darwin.urdf (robot description, URDF)
Before this commit: robot darwinOP, 31 links, 30 joints
Joints:
- joint j_gripper_l: limit lower=-2.6179939 upper=2.6179939 effort=2.8 velocity=5.6548668 -> lower=-1.24 upper=0 effort=2.8 velocity=5.6548668

Commit message: Make j_wrist_l a fixed joint
In lab we have the version with 3dof. FOr now it's ok to have this
fixed.

File: urdf/darwin.urdf (robot description, URDF)
Before this commit: robot darwinOP, 31 links, 30 joints
Joints:
- joint j_wrist_l: type revolute -> fixed

Commit message: Update lower and upper limits for j_shoulder_r (shoulder pitch)

File: urdf/darwin.urdf (robot description, URDF)
Before this commit: robot darwinOP, 31 links, 30 joints
Joints:
- joint j_shoulder_r: limit lower=-2.6179939 upper=2.6179939 effort=2.8 velocity=5.6548668 -> lower=-4.3633231 upper=4.3633231 effort=2.8 velocity=5.6548668

Commit message: Update lower and upper limits for j_high_arm_r (shoulder roll)

File: urdf/darwin.urdf (robot description, URDF)
Before this commit: robot darwinOP, 31 links, 30 joints
Joints:
- joint j_high_arm_r: limit lower=-2.6179939 upper=2.6179939 effort=2.8 velocity=5.648668 -> lower=-1.7453293 upper=1.7453293 effort=2.8 velocity=5.648668

Commit message: Update lower and upper limits for j_low_arm_r (elbow)

File: urdf/darwin.urdf (robot description, URDF)
Before this commit: robot darwinOP, 31 links, 30 joints
Joints:
- joint j_low_arm_r: limit lower=-1.635 upper=2.6179939 effort=2.8 velocity=5.6548668 -> lower=0 upper=2.7925268 effort=2.8 velocity=5.6548668

Commit message: Make j_wrist_r a fixed joint

File: urdf/darwin.urdf (robot description, URDF)
Before this commit: robot darwinOP, 31 links, 30 joints
Joints:
- joint j_wrist_r: type revolute -> fixed

Commit message: Update lower and upper limits for j_gripper_r

File: urdf/darwin.urdf (robot description, URDF)
Before this commit: robot darwinOP, 31 links, 30 joints
Joints:
- joint j_gripper_r: limit lower=-2.6179939 upper=2.6179939 effort=2.8 velocity=5.6548668 -> lower=-1.24 upper=0 effort=2.8 velocity=5.6548668

Commit message: Update lower and upper limits for j_pelvis_l (hip yaw)

File: urdf/darwin.urdf (robot description, URDF)
Before this commit: robot darwinOP, 31 links, 30 joints
Joints:
- joint j_pelvis_l: limit lower=-2.6179939 upper=2.6179939 effort=10 velocity=5.6548668 -> lower=-0.7853982 upper=2.6179939 effort=10 velocity=5.6548668

Commit message: Update lower and upper limits for j_thigh1_l (hip roll)

File: urdf/darwin.urdf (robot description, URDF)
Before this commit: robot darwinOP, 31 links, 30 joints
Joints:
- joint j_thigh1_l: limit lower=-2.6179939 upper=2.6179939 effort=10 velocity=5.6548668 -> lower=-1.0471976 upper=0 effort=10 velocity=5.6548668

Commit message: Update lower and upper limits for j_thigh2_l (hip pitch)

File: urdf/darwin.urdf (robot description, URDF)
Before this commit: robot darwinOP, 31 links, 30 joints
Joints:
- joint j_thigh2_l: limit lower=-2.6179939 upper=2.6179939 effort=10 velocity=5.6548668 -> lower=-0.5235988 upper=1.7453293 effort=10 velocity=5.6548668

Commit message: Update lower and upper limits for j_tibia_l (knee)

File: urdf/darwin.urdf (robot description, URDF)
Before this commit: robot darwinOP, 31 links, 30 joints
Joints:
- joint j_tibia_l: limit lower=-2.6179939 upper=2.6179939 effort=10 velocity=5.6548668 -> lower=-2.268928 upper=0 effort=10 velocity=5.6548668

Commit message: Update lower and upper limits for j_ankle1_l (ankle pitch)

File: urdf/darwin.urdf (robot description, URDF)
Before this commit: robot darwinOP, 31 links, 30 joints
Joints:
- joint j_ankle1_l: limit lower=-2.6179939 upper=2.6179939 effort=10 velocity=5.6548668 -> lower=-1.0471976 upper=1.0471976 effort=10 velocity=5.6548668

Commit message: Update lower and upper limits for j_ankle2_l (ankle roll)

File: urdf/darwin.urdf (robot description, URDF)
Before this commit: robot darwinOP, 31 links, 30 joints
Joints:
- joint j_ankle2_l: limit lower=-2.6179939 upper=2.6179939 effort=10 velocity=5.6548668 -> lower=-0.5235988 upper=1.0471976 effort=10 velocity=5.6548668

Commit message: Update lower and upper limits for j_pelvis_r (hip yaw)

File: urdf/darwin.urdf (robot description, URDF)
Before this commit: robot darwinOP, 31 links, 30 joints
Joints:
- joint j_pelvis_r: limit lower=-2.6179939 upper=2.6179939 effort=10 velocity=5.6548668 -> lower=-2.6179939 upper=0.7853982 effort=10 velocity=5.6548668

Commit message: Update lower and upper limits for j_thigh1_r (hip roll)

File: urdf/darwin.urdf (robot description, URDF)
Before this commit: robot darwinOP, 31 links, 30 joints
Joints:
- joint j_thigh1_r: limit lower=-2.6179939 upper=2.6179939 effort=10 velocity=5.6548668 -> lower=0 upper=1.0471976 effort=10 velocity=5.6548668

Commit message: Update lower and upper limits for j_thigh2_r (hip pitch)

File: urdf/darwin.urdf (robot description, URDF)
Before this commit: robot darwinOP, 31 links, 30 joints
Joints:
- joint j_thigh2_r: limit lower=-2.6179939 upper=2.6179939 effort=10 velocity=5.6548668 -> lower=-1.7453293 upper=0.5235988 effort=10 velocity=5.6548668

Commit message: Update lower and upper limits for j_tibia_r (knee)

File: urdf/darwin.urdf (robot description, URDF)
Before this commit: robot darwinOP, 31 links, 30 joints
Joints:
- joint j_tibia_r: limit lower=-2.6179939 upper=2.6179939 effort=10 velocity=5.6548668 -> lower=0 upper=2.268928 effort=10 velocity=5.6548668

Commit message: Update limits for j_ankle1_r (ankle pitch)

File: urdf/darwin.urdf (robot description, URDF)
Before this commit: robot darwinOP, 31 links, 30 joints
Joints:
- joint j_ankle1_r: limit lower=-2.6179939 upper=2.6179939 effort=10 velocity=5.6548668 -> lower=-1.0471976 upper=1.0471976 effort=10 velocity=5.6548668

Commit message: Update lower and upper limits for j_ankle2_r (ankle roll)

File: urdf/darwin.urdf (robot description, URDF)
Before this commit: robot darwinOP, 31 links, 30 joints
Joints:
- joint j_ankle2_r: limit lower=-2.6179939 upper=2.6179939 effort=10 velocity=5.6548668 -> lower=-0.5235988 upper=1.0471976 effort=10 velocity=5.6548668

Commit message: Put Darwin into the Zero Pose

File: urdf/darwin.urdf (robot description, URDF)
Before this commit: robot darwinOP, 31 links, 30 joints
Joints:
- joint j_ankle1_l: origin xyz=-0.093 0 0 rpy=3.14159 0 1.1388 -> xyz=-0.093 0 0 rpy=3.14159 0 0
- joint j_ankle1_r: origin xyz=0.093 0 0 rpy=3.14159 0 -1.1388 -> xyz=0.093 0 0 rpy=3.14159 0 0
- joint j_high_arm_l: origin xyz=-0.016 0 0.02165 rpy=1.5707963 0.2 0 -> xyz=-0.016 0 0.02165 rpy=1.5707963 1.5707963 0
- joint j_high_arm_r: origin xyz=0.016 0 0.02165 rpy=-1.5707963 2.9415926 0 -> xyz=0.016 0 0.02165 rpy=-1.5707963 1.5707963 0
- joint j_low_arm_l: origin xyz=-0.06 0 -0.016 rpy=-1.5707963 1.64159 0 -> xyz=-0.06 0 -0.016 rpy=-1.5707963 3.14159 0
- joint j_low_arm_r: origin xyz=-0.06 0 0.016 rpy=-1.5707963 4.64159 0 -> xyz=-0.06 0 0.016 rpy=-1.5707963 3.14159 0
- joint j_shoulder_l: origin xyz=0 0 0 rpy=0 0 -1.15 -> xyz=0 0 0 rpy=0 0 -1.5707963
- joint j_shoulder_r: origin xyz=0 0 0 rpy=0 0 -1.9907 -> xyz=0 0 0 rpy=0 0 -1.5707963
- joint j_thigh2_l: origin xyz=0 0 0 rpy=1.5707963 -1.142 -1.5707963 -> xyz=0 0 0 rpy=1.5707963 0 -1.5707963
- joint j_thigh2_r: origin xyz=0 0 0 rpy=1.5707963 1.142 -1.5707963 -> xyz=0 0 0 rpy=1.5707963 0 -1.5707963
- joint j_tibia_l: origin xyz=-0.093 0 0 rpy=0 0 -2.2788 -> xyz=-0.093 0 0 rpy=0 0 0
- joint j_tibia_r: origin xyz=0.093 0 0 rpy=0 0 2.2788 -> xyz=0.093 0 0 rpy=0 0 0

Commit message: Remove left and right gripper

File: urdf/darwin.urdf (robot description, URDF)
Before this commit: robot darwinOP, 31 links, 30 joints
Links:
- removed link MP_ARM_GRIPPER_MOV_L
- removed link MP_ARM_GRIPPER_MOV_R
Joints:
- removed joint j_gripper_l
- removed joint j_gripper_r

Commit message: Use designed arm basic low for right arm

File: urdf/darwin.urdf (robot description, URDF)
Before this commit: robot darwinOP, 29 links, 28 joints
Links:
- link MP_ARM_GRIPPER_FIX_R: geometry collision mesh filename=package://darwin_description/meshes/arm_basic_low_r.stl scale=1 1 1; visual mesh filename=package://darwin_description/meshes/arm_basic_low_r.stl scale=1 1 1

Commit message: Remove the old gripper part for right arm

File: urdf/darwin.urdf (robot description, URDF)
Before this commit: robot darwinOP, 29 links, 28 joints
Links:
- removed link MP_ARM_GRIPPER_FIX_DUMMY_R
Joints:
- removed joint j_wrist_dummy_r

Commit message: Use designed arm low left

File: urdf/darwin.urdf (robot description, URDF)
Before this commit: robot darwinOP, 28 links, 27 joints
Links:
- removed link MP_ARM_GRIPPER_FIX_DUMMY_L
- link MP_ARM_GRIPPER_FIX_L: geometry collision mesh filename=package://darwin_description/meshes/arm_basic_low_l.stl scale=1 1 1; visual mesh filename=package://darwin_description/meshes/arm_basic_low_l.stl scale=1 1 1
Joints:
- removed joint j_wrist_dummy_l

Commit message: Add a simplified body collision mesh

File: urdf/darwin.urdf (robot description, URDF)
Before this commit: robot darwinOP, 27 links, 26 joints
Links:
- link MP_BODY: geometry collision mesh filename=package://darwin_description/meshes/body_coll_simple.stl scale=1 1 1; visual mesh filename=package://darwin_description/meshes/body.STL scale=1 1 1

Commit message: Use a simplified collision mesh for the head

File: urdf/darwin.urdf (robot description, URDF)
Before this commit: robot darwinOP, 27 links, 26 joints
Links:
- link MP_HEAD: geometry collision mesh filename=package://darwin_description/meshes/head_coll_simple.stl scale=1 1 1; visual mesh filename=package://darwin_description/meshes/head.STL scale=1 1 1

Commit message: Rename head joints

File: urdf/darwin.urdf (robot description, URDF)
Before this commit: robot darwinOP, 27 links, 26 joints
Joints:
- removed joint j_pan
- removed joint j_tilt
- added joint head_pan: type revolute, parent MP_BODY, child MP_NECK, origin xyz=0 0 0.0235 rpy=0 0 1.5707963, axis 0 0 1, limit lower=-2.6179939 upper=2.6179939 effort=2.8 velocity=5.6548668
- added joint head_tilt: type revolute, parent MP_NECK, child MP_HEAD, origin xyz=0 0 0.02715 rpy=-1.5707963 0 1.5707963, axis 0 0 1, limit lower=-1.0471976 upper=0.5235988 effort=2.8 velocity=5.6548668

Commit message: Update joints name for left shoulder

File: urdf/darwin.urdf (robot description, URDF)
Before this commit: robot darwinOP, 27 links, 26 joints
Joints:
- removed joint j_high_arm_l
- removed joint j_shoulder_l
- added joint l_sho_pitch: type revolute, parent MP_BACK_L, child MP_SHOULDER_L, origin xyz=0 0 0 rpy=0 0 -1.5707963, axis 0 0 1, limit lower=-4.3633231 upper=4.3633231 effort=2.8 velocity=5.6548668
- added joint l_sho_roll: type revolute, parent MP_SHOULDER_L, child MP_ARM_HIGH_L, origin xyz=-0.016 0 0.02165 rpy=1.5707963 1.5707963 0, axis 0 0 1, limit lower=-1.7453293 upper=1.7453293 effort=2.8 velocity=5.648668

Commit message: Update name for left elbow joint

File: urdf/darwin.urdf (robot description, URDF)
Before this commit: robot darwinOP, 27 links, 26 joints
Joints:
- removed joint j_low_arm_l
- added joint l_el: type revolute, parent MP_ARM_HIGH_L, child MP_ARM_LOW_L, origin xyz=-0.06 0 -0.016 rpy=-1.5707963 3.14159 0, axis 0 0 1, limit lower=-2.7925268 upper=0 effort=2.8 velocity=5.6548668

Commit message: Update right arm joints name

File: urdf/darwin.urdf (robot description, URDF)
Before this commit: robot darwinOP, 27 links, 26 joints
Joints:
- removed joint j_high_arm_r
- removed joint j_low_arm_r
- removed joint j_shoulder_r
- added joint r_el: type revolute, parent MP_ARM_HIGH_R, child MP_ARM_LOW_R, origin xyz=-0.06 0 0.016 rpy=-1.5707963 3.14159 0, axis 0 0 1, limit lower=0 upper=2.7925268 effort=2.8 velocity=5.6548668
- added joint r_sho_pitch: type revolute, parent MP_BACK_R, child MP_SHOULDER_R, origin xyz=0 0 0 rpy=0 0 -1.5707963, axis 0 0 1, limit lower=-4.3633231 upper=4.3633231 effort=2.8 velocity=5.6548668
- added joint r_sho_roll: type revolute, parent MP_SHOULDER_R, child MP_ARM_HIGH_R, origin xyz=0.016 0 0.02165 rpy=-1.5707963 1.5707963 0, axis 0 0 1, limit lower=-1.7453293 upper=1.7453293 effort=2.8 velocity=5.648668

Commit message: Update joint name for hip yaw

File: urdf/darwin.urdf (robot description, URDF)
Before this commit: robot darwinOP, 27 links, 26 joints
Joints:
- removed joint j_pelvis_l
- added joint l_hip_yaw: type revolute, parent MP_BODY, child MP_PELVIS_L, origin xyz=-0.005 0.037 -0.09355 rpy=0 3.14159 -1.5707963, axis 0 0 1, limit lower=-0.7853982 upper=2.6179939 effort=10 velocity=5.6548668

Commit message: Rename hip roll joint

File: urdf/darwin.urdf (robot description, URDF)
Before this commit: robot darwinOP, 27 links, 26 joints
Joints:
- removed joint j_thigh1_l
- added joint l_hip_roll: type revolute, parent MP_PELVIS_L, child MP_THIGH1_L, origin xyz=0 0 0.028652 rpy=1.5707963 0 0, axis 0 0 1, limit lower=-1.0471976 upper=0 effort=10 velocity=5.6548668

Commit message: Update name for hip pitch joint

File: urdf/darwin.urdf (robot description, URDF)
Before this commit: robot darwinOP, 27 links, 26 joints
Joints:
- removed joint j_thigh2_l
- added joint l_hip_pitch: type revolute, parent MP_THIGH1_L, child MP_THIGH2_L, origin xyz=0 0 0 rpy=1.5707963 0 -1.5707963, axis 0 0 1, limit lower=-0.5235988 upper=1.7453293 effort=10 velocity=5.6548668

Commit message: Update name for left knee

File: urdf/darwin.urdf (robot description, URDF)
Before this commit: robot darwinOP, 27 links, 26 joints
Joints:
- removed joint j_tibia_l
- added joint l_knee: type revolute, parent MP_THIGH2_L, child MP_TIBIA_L, origin xyz=-0.093 0 0 rpy=0 0 0, axis 0 0 1, limit lower=-2.268928 upper=0 effort=10 velocity=5.6548668

Commit message: Rename ankle left pitch

File: urdf/darwin.urdf (robot description, URDF)
Before this commit: robot darwinOP, 27 links, 26 joints
Joints:
- removed joint j_ankle1_l
- added joint l_ank_pitch: type revolute, parent MP_TIBIA_L, child MP_ANKLE1_L, origin xyz=-0.093 0 0 rpy=3.14159 0 0, axis 0 0 1, limit lower=-1.0471976 upper=1.0471976 effort=10 velocity=5.6548668

Commit message: Rename ankle roll joint

File: urdf/darwin.urdf (robot description, URDF)
Before this commit: robot darwinOP, 27 links, 26 joints
Joints:
- removed joint j_ankle2_l
- added joint l_ank_roll: type revolute, parent MP_ANKLE1_L, child MP_ANKLE2_L, origin xyz=0 0 0 rpy=-1.5707963 0 0, axis 0 0 1, limit lower=-0.5235988 upper=1.0471976 effort=10 velocity=5.6548668
