Commit message: Update right leg joints name

File: urdf/darwin.urdf (robot description, URDF)
Before this commit: robot darwinOP, 27 links, 26 joints
Joints:
- removed joint j_ankle1_r
- removed joint j_ankle2_r
- removed joint j_pelvis_r
- removed joint j_thigh1_r
- removed joint j_thigh2_r
- removed joint j_tibia_r
- added joint r_ank_pitch: type revolute, parent MP_TIBIA_R, child MP_ANKLE1_R, origin xyz=0.093 0 0 rpy=3.14159 0 0, axis 0 0 1, limit lower=-1.0471976 upper=1.0471976 effort=10 velocity=5.6548668
- added joint r_ank_roll: type revolute, parent MP_ANKLE1_R, child MP_ANKLE2_R, origin xyz=0 0 0 rpy=-1.5707963 0 0, axis 0 0 1, limit lower=-0.5235988 upper=1.0471976 effort=10 velocity=5.6548668
- added joint r_hip_pitch: type revolute, parent MP_THIGH1_R, child MP_THIGH2_R, origin xyz=0 0 0 rpy=1.5707963 0 -1.5707963, axis 0 0 1, limit lower=-1.7453293 upper=0.5235988 effort=10 velocity=5.6548668
- added joint r_hip_roll: type revolute, parent MP_PELVIS_R, child MP_THIGH1_R, origin xyz=0 0 0.028652 rpy=-1.5707963 0 0, axis 0 0 1, limit lower=0 upper=1.0471976 effort=10 velocity=5.6548668
- added joint r_hip_yaw: type revolute, parent MP_BODY, child MP_PELVIS_R, origin xyz=-0.005 -0.037 -0.09355 rpy=0 3.14159 1.5707963, axis 0 0 1, limit lower=-2.6179939 upper=0.7853982 effort=10 velocity=5.6548668
- added joint r_knee: type revolute, parent MP_THIGH2_R, child MP_TIBIA_R, origin xyz=0.093 0 0 rpy=0 0 0, axis 0 0 1, limit lower=0 upper=2.268928 effort=10 velocity=5.6548668

Commit message: Revert "Add a simplified body collision mesh"
This reverts commit cffa22b545612c79a04772414a19e1afa82c92be.

File: urdf/darwin.urdf (robot description, URDF)
Before this commit: robot darwinOP, 27 links, 26 joints
Links:
- link MP_BODY: geometry collision mesh filename=package://darwin_description/meshes/body_coll.stl scale=1 1 1; visual mesh filename=package://darwin_description/meshes/body.STL scale=1 1 1
